File: n64-kicad/n64-kicad.kicad_sch (KiCad schematic)
At the start: 0 parts

Commit message: Rename files
Other:
- sheet NUS-CPU-(P)-01 renamed NUS-CPU(P)-01
- sheet NUS-CPU-(P)-01-PicoDVI renamed NUS-CPU(P)-01-PicoDVI
- added sheet NUS-CPU-03 (NUS-CPU-03.kicad_sch)
- sheet NUS-CPU(P)-01: file NUS-CPU-(P)-01.kicad_sch -> NUS-CPU(P)-01.kicad_sch
- sheet NUS-CPU(P)-01-PicoDVI: file NUS-CPU-(P)-01-PicoDVI.kicad_sch -> NUS-CPU(P)-01-PicoDVI.kicad_sch
- note added: "Hardware Mod wiring guides"
- note added: "NTSC versions"
- note added: "NUS-CPU(R)-01 NUS-CPU(P)-01 NUS-CPU(P)-02 NUS-CPU(P)-03 NUS-CPU(P)-03-1"
- note added: "NUS-CPU-01 NUS-CPU-02 NUS-CPU-03 NUS-CPU-04 NUS-CPU-05 NUS-CPU-05-01 NUS-CPU-06 NUS-CPU-07 NUS-CPU-08 NUS-CPU-08-1 NUS-CPU-09 NUS-CPU-09-1"
- note added: "PAL versions"
Changed lines of the file:
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@@
 (kicad_sch (version 20230121) (generator eeschema)
   (paper "A4")
-  (sheet (at 38.1 43.18) (size 12.7 5.08) (fields_autoplaced)
+  (text "NTSC versions" (at 39.37 24.13 0)
+    (effects (font (size 2.54 2.54)) (justify left bottom))
+  )
+  (text "NUS-CPU-01\nNUS-CPU-02\nNUS-CPU-03\nNUS-CPU-04\nNUS-CPU-05\nNUS-CPU-05-01\nNUS-CPU-06\nNUS-CPU-07\nNUS-CPU-08\nNUS-CPU-08-1\nNUS-CPU-09\nNUS-CPU-09-1"
+    (at 39.37 50.8 0)
+    (effects (font (size 1.27 1.27)) (justify left bottom))
+  )
+  (text "Hardware Mod wiring guides" (at 38.1 95.25 0)
+    (effects (font (size 2.54 2.54)) (justify left bottom))
+  )
+  (text "PAL versions" (at 90.17 25.4 0)
+    (effects (font (size 2.54 2.54)) (justify left bottom))
+  )
+  (text "NUS-CPU(R)-01\nNUS-CPU(P)-01\nNUS-CPU(P)-02\nNUS-CPU(P)-03\nNUS-CPU(P)-03-1"
+    (at 90.17 36.83 0)
+    (effects (font (size 1.27 1.27)) (justify left bottom))
+  )
+  (sheet (at 39.37 101.6) (size 12.7 5.08) (fields_autoplaced)
     (stroke (width 0.1524) (type solid))
     (fill (color 0 0 0 0.0000))
-    (property "Sheetname" "NUS-CPU-(P)-01-PicoDVI" (at 38.1 42.4684 0)
+    (property "Sheetname" "NUS-CPU(P)-01-PicoDVI" (at 39.37 100.8884 0)
       (effects (font (size 1.27 1.27)) (justify left bottom))
     )
-    (property "Sheetfile" "NUS-CPU-(P)-01-PicoDVI.kicad_sch" (at 38.1 48.8446 0)
+    (property "Sheetfile" "NUS-CPU(P)-01-PicoDVI.kicad_sch" (at 39.37 107.2646 0)
       (effects (font (size 1.27 1.27)) (justify left top))
     )
-    (property "Field2" "" (at 38.1 43.18 0)
+    (property "Field2" "" (at 39.37 101.6 0)
       (effects (font (size 1.27 1.27)) hide)
     )
@@
     )
   )
-  (sheet (at 38.1 25.4) (size 12.7 5.08) (fields_autoplaced)
+  (sheet (at 90.17 63.5) (size 12.7 5.08) (fields_autoplaced)
     (stroke (width 0.1524) (type solid))
     (fill (color 0 0 0 0.0000))
-    (property "Sheetname" "NUS-CPU-(P)-01" (at 38.1 24.6884 0)
+    (property "Sheetname" "NUS-CPU(P)-01" (at 90.17 62.7884 0)
       (effects (font (size 1.27 1.27)) (justify left bottom))
     )
-    (property "Sheetfile" "NUS-CPU-(P)-01.kicad_sch" (at 38.1 31.0646 0)
+    (property "Sheetfile" "NUS-CPU(P)-01.kicad_sch" (at 90.17 69.1646 0)
       (effects (font (size 1.27 1.27)) (justify left top))
+    )
+    (property "Field2" "" (at 90.17 63.5 0)
+      (effects (font (size 1.27 1.27)) hide)
     )
     (instances
@@
       )
     )
+  )
+  (sheet (at 39.37 63.5) (size 12.7 5.08) (fields_autoplaced)
+    (stroke (width 0.1524) (type solid))
+    (fill (color 0 0 0 0.0000))
+    (property "Sheetname" "NUS-CPU-03" (at 39.37 62.7884 0)
+      (effects (font (size 1.27 1.27)) (justify left bottom))
+    )
+    (property "Sheetfile" "NUS-CPU-03.kicad_sch" (at 39.37 69.1646 0)
+      (effects (font (size 1.27 1.27)) (justify left top))
+    )
+    (property "Field2" "" (at 39.37 63.5 0)
+      (effects (font (size 1.27 1.27)) hide)
+    )
+    (instances
+      (project "n64-kicad"
+        (path "/62362fc5-d8b0-453c-8cf3-9bf5adb1c5ec" (page "4"))
+      )
+    )
